File: CAD/uplc/uplc.kicad_pcb (KiCad board)
At the start: 4 copper layers, 31.2 x 20.5 mm, 46 parts, among them J1 Conn_01x06_Pin, J2 SM12B-GHS-TB(LF)(SN), K1 G6K-2F-Y, K2 G6K-2F-Y, U1 DS8242-33S5, U3 ESP32-C3-WROOM-02, U5 TBD62003AFWG, Y1 32.568khz

Commit message: wip
Parts:
- removed the D2 at (124.2, 76.5)
- removed kibuzzard-65666C6B: G***, esprelay:kibuzzard-65666C6B
- removed kibuzzard-65666C71: G***, esprelay:kibuzzard-65666C71
- removed kibuzzard-65666C76: G***, esprelay:kibuzzard-65666C76
- removed kibuzzard-65666C7B: G***, esprelay:kibuzzard-65666C7B
- removed kibuzzard-65666C87: G***, esprelay:kibuzzard-65666C87
- removed kibuzzard-65666CB7: G***, esprelay:kibuzzard-65666CB7
- removed kibuzzard-65CFDA91: G***, esprelay:kibuzzard-65CFDA91
- removed kibuzzard-65CFDAA0: G***, esprelay:kibuzzard-65CFDAA0
- removed kibuzzard-65CFDAA7: G***, esprelay:kibuzzard-65CFDAA7
- removed kibuzzard-65CFDAAD: G***, esprelay:kibuzzard-65CFDAAD
- removed kibuzzard-65CFDAB5: G***, esprelay:kibuzzard-65CFDAB5
- removed kibuzzard-65CFDABC: G***, esprelay:kibuzzard-65CFDABC
- added C6: 0.1uF, Capacitor_SMD:C_0402_1005Metric, F.Cu at (106.6, 73.5)
- added D3: 1N5819WS, Diode_SMD:D_SOD-323, F.Cu at (124.2, 76.5)
- added kibuzzard-65D3605C: G***, kibuzzard-65D3605C, F.Cu at (104.4, 82.6)
- added kibuzzard-65D3616E: G***, kibuzzard-65D3616E, B.Cu at (128.0, 74.0)
- added kibuzzard-65D36177: G***, kibuzzard-65D36177, B.Cu at (128.0, 75.6)
- added kibuzzard-65D3619D: G***, kibuzzard-65D3619D, B.Cu at (128.0, 78.7)
- added kibuzzard-65D361A7: G***, kibuzzard-65D361A7, B.Cu at (128.0, 77.1)
- added kibuzzard-65D361B0: G***, kibuzzard-65D361B0, B.Cu at (128.0, 80.2)
- added kibuzzard-65D361D3: G***, kibuzzard-65D361D3, B.Cu at (128.0, 81.8)
- added kibuzzard-65D361E1: G***, kibuzzard-65D361E1, B.Cu at (128.0, 83.3)
- added kibuzzard-65D361E9: G***, kibuzzard-65D361E9, B.Cu at (128.0, 84.9)
- added kibuzzard-65D361F2: G***, kibuzzard-65D361F2, B.Cu at (128.0, 86.4)
- added kibuzzard-65D361FD: G***, kibuzzard-65D361FD, B.Cu at (128.0, 88.0)
- added kibuzzard-65D36206: G***, kibuzzard-65D36206, B.Cu at (128.0, 89.5)
- added kibuzzard-65D3620E: G***, kibuzzard-65D3620E, B.Cu at (128.0, 91.1)
- added kibuzzard-65D36263: G***, kibuzzard-65D36263, B.Cu at (123.5, 86.1)
- added kibuzzard-65D36263: G***, kibuzzard-65D36263, B.Cu at (123.6, 78.4)
- added kibuzzard-65D36263: G***, kibuzzard-65D36263, B.Cu at (123.5, 75.9)
- added kibuzzard-65D36263: G***, kibuzzard-65D36263, B.Cu at (123.6, 83.5)
- added kibuzzard-65D36263: G***, kibuzzard-65D36263, B.Cu at (123.5, 88.6)
- added kibuzzard-65D36263: G***, kibuzzard-65D36263, B.Cu at (123.7, 81.0)
- C1, C4: value 10pf -> 20pf
- D1, D2: value 1N4148WS -> 1N5819WS
- moved C3 1.15 mm to (111.1, 73.5), turned to 90 degrees
- moved C10 1.03 mm to (110.0, 73.5)
- moved R2 0.99 mm to (123.8, 80.9)
- moved R1 0.97 mm to (124.7, 80.9)
- moved C11 0.92 mm to (108.9, 73.5)
- moved R5 0.78 mm to (107.8, 73.5)
- moved R11 0.77 mm to (112.3, 73.5)
- moved C2 0.75 mm to (123.8, 74.4)
- moved C5 0.75 mm to (121.7, 74.4)
- moved R12 0.67 mm to (113.4, 73.5)
- moved J1 0.59 mm to (121.2, 75.9)
- moved R10 0.56 mm to (114.6, 73.5)
- moved R9 0.46 mm to (115.7, 73.5)
- moved R4 0.35 mm to (116.9, 73.5)
- moved R3 0.35 mm to (120.3, 73.5), turned to -90 degrees
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Connections:
- J1 pad 2: TX -> GND
- J1 pad 3: RX -> BOOT
- J1 pad 4: BOOT -> RST
- J1 pad 5: RST -> TX
- J1 pad 6: GND -> RX
- J2 pad 1: +VDC -> R2NO
- J2 pad 10: R2NC -> HO1
- J2 pad 11: R2CO -> GND
- J2 pad 12: R2NO -> +VDC
- J2 pad 2: GND -> R2CO
- J2 pad 3: HI1 -> R2NC
- J2 pad 4: HI2 -> R1NO
- J2 pad 5: HO1 -> R1CO
- J2 pad 6: HO2 -> R1NC
- J2 pad 7: R1NC -> HI2
- J2 pad 8: R1CO -> HI1
- J2 pad 9: R1NO -> HO2
- R10 pad 1: GPIO15 -> LI5
- R7 pad 1: GPIO13 -> LI12
- R8 pad 1: GPIO12 -> LI3
- R9 pad 1: GPIO14 -> LI4
- U3 pad 10: GPIO15 -> unconnected-(U3-GPIO10-Pad10)
- U3 pad 13: unconnected-(U3-GPIO18/USB_D--Pad13) -> LO6
- U3 pad 14: GPIO4 -> LO7
- U3 pad 15: ADC -> LI3
- U3 pad 3: GPIO5 -> ADC
- U3 pad 4: GPIO12 -> LI4
- U3 pad 5: GPIO13 -> LI5
- U3 pad 6: GPIO14 -> LI12
- U5 pad 1: GPIO13 -> LI12
- U5 pad 10: GPIO5 -> LO7
- U5 pad 11: GPIO4 -> LO6
- U5 pad 12: RO2 -> RO1
- U5 pad 13: RO1 -> RO2
- U5 pad 2: GPIO13 -> LI12
- U5 pad 3: GPIO12 -> LI3
- U5 pad 4: GPIO14 -> LI4
- U5 pad 5: GPIO15 -> LI5
Routing:
- net +3.3V: track 0.00 -> 63.7 mm, vias 0 -> 10
- net GND: track 0.00 -> 50.1 mm, vias 0 -> 55
- net R1NO: track 0.00 -> 28.5 mm
- net RST: track 0.00 -> 27.3 mm, vias 0 -> 2
- net LI3: track 0.00 -> 24.2 mm, vias 0 -> 1
- net HI2: track 0.00 -> 24.1 mm, vias 0 -> 2
- net HI1: track 0.00 -> 22.0 mm, vias 0 -> 2
- net R1CO: track 0.00 -> 21.8 mm
- net R1NC: track 0.00 -> 21.1 mm
- net ADC: track 2.62 -> 23.1 mm, vias 0 -> 3
- net Net-(U3-GPIO2/ADC1_CH2): track 0.00 -> 18.7 mm, vias 0 -> 1
- net Net-(U3-GPIO1/ADC1_CH1/XTAL_32K_N): track 0.00 -> 18.3 mm, vias 0 -> 1
- net HO2: track 0.00 -> 17.1 mm, vias 0 -> 4
- net HO1: track 0.00 -> 16.6 mm, vias 0 -> 4
- net Net-(U3-GPIO0/ADC1_CH0/XTAL_32K_P): track 0.00 -> 16.1 mm, vias 0 -> 1
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- added copper zone on F.Cu, net +3.3V
- added copper zone on In2.Cu, net +3.3V
- added copper zone on In1.Cu, net GND
- added copper zone on In2.Cu, net GND
- added copper zone on In2.Cu, net HO1
- added copper zone on In2.Cu, net HO2
Other:
- board size 31.2 x 20.5 mm -> 31.1 x 21 mm

Commit message: Rev 1.0
Parts:
- removed kibuzzard-65D272D8: G***, kibuzzard-65D272D8
- removed kibuzzard-65D3605C: G***, kibuzzard-65D3605C
- removed kibuzzard-65D36263 (x6): G***, kibuzzard-65D36263
- added kibuzzard-65D45F97: G***, esprelay:kibuzzard-65D45F97, B.Cu at (123.6, 76.0)
- added kibuzzard-65D45FF4: G***, esprelay:kibuzzard-65D45FF4, B.Cu at (123.7, 78.4)
- added kibuzzard-65D4601A: G***, esprelay:kibuzzard-65D4601A, B.Cu at (123.7, 81.0)
- added kibuzzard-65D46022: G***, esprelay:kibuzzard-65D46022, B.Cu at (123.7, 83.7)
- added kibuzzard-65D46066: G***, esprelay:kibuzzard-65D46066, B.Cu at (123.7, 86.1)
- added kibuzzard-65D460A0: G***, esprelay:kibuzzard-65D460A0, B.Cu at (123.7, 88.6)
- added kibuzzard-65D4907E: G***, kibuzzard-65D4907E, F.Cu at (104.5, 82.6)
- added kibuzzard-65D49092: G***, kibuzzard-65D49092, F.Cu at (101.8, 82.6)
- U3: footprint Espressif:ESP32-C3-WROOM-02 -> PCM_Espressif:ESP32-C3-WROOM-02
- kibuzzard-65D3616E: footprint kibuzzard-65D3616E -> esprelay:kibuzzard-65D3616E
- kibuzzard-65D36177: footprint kibuzzard-65D36177 -> esprelay:kibuzzard-65D36177
- kibuzzard-65D3619D: footprint kibuzzard-65D3619D -> esprelay:kibuzzard-65D3619D
- kibuzzard-65D361A7: footprint kibuzzard-65D361A7 -> esprelay:kibuzzard-65D361A7
- kibuzzard-65D361B0: footprint kibuzzard-65D361B0 -> esprelay:kibuzzard-65D361B0
- kibuzzard-65D361D3: footprint kibuzzard-65D361D3 -> esprelay:kibuzzard-65D361D3
- kibuzzard-65D361E1: footprint kibuzzard-65D361E1 -> esprelay:kibuzzard-65D361E1
- kibuzzard-65D361E9: footprint kibuzzard-65D361E9 -> esprelay:kibuzzard-65D361E9
- kibuzzard-65D361F2: footprint kibuzzard-65D361F2 -> esprelay:kibuzzard-65D361F2
- kibuzzard-65D361FD: footprint kibuzzard-65D361FD -> esprelay:kibuzzard-65D361FD
- kibuzzard-65D36206: footprint kibuzzard-65D36206 -> esprelay:kibuzzard-65D36206
- kibuzzard-65D3620E: footprint kibuzzard-65D3620E -> esprelay:kibuzzard-65D3620E
- moved kibuzzard-65D3616E 0.40 mm to (128.4, 74.0)
- moved kibuzzard-65D36177 0.40 mm to (128.4, 75.6)
- moved kibuzzard-65D3619D 0.40 mm to (128.4, 78.7)
- moved kibuzzard-65D361A7 0.40 mm to (128.4, 77.1)
- moved kibuzzard-65D361B0 0.40 mm to (128.4, 80.2)
- moved kibuzzard-65D361D3 0.40 mm to (128.4, 81.8)
- moved kibuzzard-65D361E1 0.40 mm to (128.4, 83.3)
- moved kibuzzard-65D361E9 0.40 mm to (128.4, 84.9)
- moved kibuzzard-65D361F2 0.40 mm to (128.4, 86.4)
- moved kibuzzard-65D361FD 0.40 mm to (128.4, 88.0)
- moved kibuzzard-65D36206 0.40 mm to (128.4, 89.5)
- moved kibuzzard-65D3620E 0.40 mm to (128.4, 91.1)
Routing:
- net +3.3V: track 63.7 -> 73.2 mm
- net GND: track 50.1 -> 54.2 mm
- net RST: track 27.3 -> 25.8 mm
- net RO1: track 9.48 -> 8.21 mm
- net LI3: track 24.2 -> 23.0 mm
- net LO6: track 15.4 -> 14.4 mm
- net Net-(U3-GPIO8): track 7.63 -> 6.56 mm
- net R2NO: track 11.2 -> 10.4 mm
- net Net-(U3-GPIO1/ADC1_CH1/XTAL_32K_N): track 18.3 -> 17.7 mm
- net R1CO: track 21.8 -> 21.3 mm
Other:
- outline, holes or cut-outs redrawn
- board text removed: "3v3"
- board text removed: "boot"
- board text removed: "gnd"
- board text removed: "rst"
- board text removed: "rxd"
- board text removed: "txd"

Commit message: Value updates
Parts:
- Y1: value 32.568khz -> 32.568khz 3.2x1.5 12.5pf
Changed lines of the file:
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@@
       (net 1 "+VDC") (pinfunction "Pin_12") (pintype "passive"))
     (pad "MP" smd roundrect (at -8.725 1.35 90) (size 1 2.7) (layers "F.Cu" "F.Paste" "F.Mask") (roundrect_rratio 0.25)
-      (net 2 "GND") (pinfunction "Pin_13") (pintype "passive"))
+      (net 2 "GND") (pinfunction "Pin_14") (pintype "passive"))
     (pad "MP" smd roundrect (at 8.725 1.35 90) (size 1 2.7) (layers "F.Cu" "F.Paste" "F.Mask") (roundrect_rratio 0.25)
-      (net 2 "GND") (pinfunction "Pin_13") (pintype "passive"))
+      (net 2 "GND") (pinfunction "Pin_14") (pintype "passive"))
     (model "${KICAD7_3DMODEL_DIR}/Connector_JST.3dshapes/JST_GH_SM12B-GHS-TB_1x12-1MP_P1.25mm_Horizontal.wrl"
       (offset (xyz 0 0 0))
@@
         (effects (font (size 1 1) (thickness 0.15)))
     )
-    (fp_text value "32.568khz" (at 0 2 90) (layer "F.Fab") hide
+    (fp_text value "32.568khz 3.2x1.5 12.5pf" (at 0 2 90) (layer "F.Fab") hide
         (effects (font (size 1 1) (thickness 0.15)))
     )
@@
     (descr "ESP32-C3-WROOM-02: https://www.espressif.com/sites/default/files/documentation/esp32-c3-wroom-02_datasheet_en.pdf")
     (tags "ESP32-C3")
+    (property "LCSC Part #" "C2934560")
     (property "Sheetfile" "uplc.kicad_sch")
     (property "Sheetname" "")

Commit message: rev 1.1
Parts:
- removed U5: TBD62003AFWG, Package_SO:SOIC-16_3.9x9.9mm_P1.27mm
- removed kibuzzard-65D45F97: G***, esprelay:kibuzzard-65D45F97
- removed kibuzzard-65D45FF4: G***, esprelay:kibuzzard-65D45FF4
- removed kibuzzard-65D4601A: G***, esprelay:kibuzzard-65D4601A
- removed kibuzzard-65D4907E: G***, kibuzzard-65D4907E
- added C12: 22uf, Capacitor_SMD:C_0402_1005Metric, F.Cu at (120.2, 79.8)
- added C8: 22uf, Capacitor_SMD:C_0402_1005Metric, F.Cu at (119.2, 79.8)
- added D4: 1N5819WS, Diode_SMD:D_SOD-323, F.Cu at (122.2, 73.7)
- added L1: 6.8uH, Inductor_SMD:L_1008_2520Metric, F.Cu at (122.6, 80.5)
- added R14: 182k, Resistor_SMD:R_0402_1005Metric, F.Cu at (124.1, 74.5)
- added R15: 62k, Resistor_SMD:R_0402_1005Metric, F.Cu at (124.6, 76.0)
- added U2: ULN2803QN, Package_DFN_QFN:QFN-20-1EP_4x4mm_P0.5mm_EP2.6x2.6mm, F.Cu at (112.8, 77.8)
- added kibuzzard-65D60D86: G***, kibuzzard-65D60D86, F.Cu at (104.5, 82.6)
- C11: value 1uF -> 22uf
- C2: value 1uF -> 0.1uF
- C5: value 0.1uF -> 4.7uF; footprint Capacitor_SMD:C_0402_1005Metric -> Capacitor_SMD:C_0603_1608Metric
- C7: value 1uF -> 4.7uF; footprint Capacitor_SMD:C_0402_1005Metric -> Capacitor_SMD:C_0603_1608Metric
- U1: value DS8242-33S5 -> AP63201WU; footprint Package_TO_SOT_SMD:SOT-23-5 -> Package_TO_SOT_SMD:TSOT-23-6
- moved R1 18.7 mm to (107.6, 73.5)
- moved R5 11.8 mm to (119.6, 73.5)
- moved R2 9.10 mm to (118.6, 73.5)
- moved D3 7.52 mm to (116.7, 77.4)
- moved C9 6.17 mm to (124.0, 73.5)
- moved R6 4.58 mm to (119.8, 75.4)
- moved D2 4.57 mm to (117.1, 81.1), turned to 180 degrees
- moved C2 3.89 mm to (124.6, 78.2), turned to 90 degrees
- moved C5 3.48 mm to (119.9, 77.3), turned to -90 degrees
- moved C7 3.29 mm to (118.4, 77.3), turned to -90 degrees
- moved R3 3.03 mm to (117.9, 75.4), turned to 180 degrees
- moved R7 2.54 mm to (116.6, 73.5)
- moved R8 2.40 mm to (115.6, 73.5)
- moved R9 1.11 mm to (114.6, 73.5)
- moved R10 0.96 mm to (113.6, 73.5)
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Connections:
- C2 pad 1: +VDC -> /SW
- C2 pad 2: GND -> Net-(U1-BST)
- C5 pad 1: GND -> /VIN_P
- C5 pad 2: +VDC -> GND
- C7 pad 1: +3.3V -> /VIN_P
- C9 pad 2: GND -> /FB
- R6 pad 1: +VDC -> /VIN_P
- U1 pad 1: +VDC -> /FB
- U1 pad 2: GND -> /VIN_P
- U1 pad 3: unconnected-(U1-NC-Pad3) -> /VIN_P
- U1 pad 4: unconnected-(U1-NC-Pad4) -> GND
- U1 pad 5: +3.3V -> /SW
- U3 pad 4: LI4 -> LI5
- U3 pad 5: LI5 -> LI4
Routing:
- net Net-(U3-GPIO2/ADC1_CH2): track 18.4 -> 37.5 mm, vias 1 -> 3
- net GND: track 54.2 -> 42.0 mm, vias 55 -> 47
- net ADC: track 22.6 -> 11.9 mm, vias 3 -> 1
- net +3.3V: track 73.2 -> 78.8 mm, vias 10 -> 12
- net /VIN_P: track 0.00 -> 5.02 mm
- net /SW: track 0.00 -> 4.99 mm
- net LI4: track 9.38 -> 4.41 mm
- net LI12: track 11.4 -> 6.85 mm
- net HI1: track 21.9 -> 26.0 mm
- net Net-(U3-GPIO8): track 6.56 -> 2.75 mm
- net /FB: track 0.00 -> 3.47 mm
- net HI2: track 24.1 -> 27.2 mm
- net +VDC: track 8.82 -> 6.74 mm
- net LI5: track 6.36 -> 4.35 mm
- net RO1: track 8.21 -> 10.0 mm
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- added copper zone on F.Cu, net /VIN_P

Commit message: Rev 1.2
Parts:
- removed C10, C6: 0.1uF, Capacitor_SMD:C_0402_1005Metric
- removed C7: 4.7uF, Capacitor_SMD:C_0603_1608Metric
- removed D3: 1N5819WS, Diode_SMD:D_SOD-323
- removed R13: 1M, Resistor_SMD:R_0402_1005Metric
- removed R3: 13.7k, Resistor_SMD:R_0402_1005Metric
- removed R6: 316k, Resistor_SMD:R_0402_1005Metric
- removed kibuzzard-65D60D86: G***, kibuzzard-65D60D86
- added kibuzzard-65D6FF37: G***, kibuzzard-65D6FF37, F.Cu at (104.5, 82.6)
- C5: value 4.7uF -> 10uF; footprint Capacitor_SMD:C_0603_1608Metric -> Capacitor_SMD:C_0805_2012Metric
- U2: value ULN2803QN -> TBD62003AFWG; footprint Package_DFN_QFN:QFN-20-1EP_4x4mm_P0.5mm_EP2.6x2.6mm -> Package_SO:SOIC-16_3.9x9.9mm_P1.27mm
- moved C3 3.83 mm to (106.8, 73.2)
- moved D2 3.14 mm to (120.2, 80.7), turned to -90 degrees
- moved R10 2.82 mm to (110.8, 73.2)
- moved C9 2.09 mm to (126.1, 73.4), turned to -90 degrees
- moved C1 2.08 mm to (107.1, 80.0), turned to 0 degrees
- moved C4 2.00 mm to (107.0, 75.2), turned to 180 degrees
- moved C5 1.83 mm to (120.2, 75.5)
- moved C8 1.71 mm to (119.8, 78.1)
- moved C12 1.70 mm to (120.7, 78.1)
- moved R14 1.50 mm to (125.1, 73.4), turned to 90 degrees
- moved L1 1.32 mm to (123.5, 79.5)
- moved U1 1.28 mm to (122.9, 75.9)
- moved U2 1.22 mm to (114.0, 78.2)
- moved R1 1.17 mm to (108.8, 73.2)
- moved C2 1.17 mm to (125.1, 77.1)
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Connections:
- U2 pad 1: LI3 -> LI12
- U2 pad 10: LO7 -> RO1
- U2 pad 11: LO6 -> LO7
- U2 pad 12: RO1 -> LO6
- U2 pad 15: HO2 -> HO1
- U2 pad 2: LI3 -> LI12
- U2 pad 3: LI4 -> LI3
- U2 pad 4: LI5 -> LI4
- U2 pad 7: (no net) -> LI5
Routing:
- net +3.3V: track 78.8 -> 11.5 mm, vias 12 -> 2
- net GND: track 42.0 -> 0.00 mm, vias 47 -> 0
- net HI2: track 27.2 -> 2.16 mm, vias 2 -> 0
- net HI1: track 26.0 -> 2.28 mm, vias 2 -> 0
- net LI3: track 23.3 -> 4.04 mm
- net HO2: track 18.8 -> 0.00 mm, vias 4 -> 0
- net HO1: track 17.0 -> 0.00 mm, vias 4 -> 0
- net ADC: track 11.9 -> 0.00 mm, vias 1 -> 0
- net TX: track 7.88 -> 0.00 mm
- net +VDC: track 6.74 -> 0.00 mm
- net RX: track 5.44 -> 0.00 mm
- net /VIN_P: track 5.02 -> 0.00 mm
- net /SW: track 4.99 -> 0.00 mm
- net LI4: track 4.41 -> 8.07 mm
- net /FB: track 3.47 -> 0.00 mm
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- removed copper zone on F.Cu, net +3.3V
- removed copper zone on F.Cu, net /VIN_P
Other:
- board size 31.1 x 21 mm -> 31.4 x 21 mm

Commit message: Production push rev 1.2
Parts:
- added kibuzzard-65D7176D: G***, kibuzzard-65D7176D, B.Cu at (123.8, 81.0)
- added kibuzzard-65D71774: G***, kibuzzard-65D71774, B.Cu at (123.8, 78.5)
- added kibuzzard-65D7177B: G***, kibuzzard-65D7177B, B.Cu at (123.8, 76.1)
- Y1: value 32.568khz 3.2x1.5 12.5pf -> 32.768khz 3215 12.5pf
- moved R4 0.98 mm to (115.7, 73.2)
- moved R7 0.98 mm to (116.6, 73.2)
- moved kibuzzard-65D46022 0.40 mm to (123.7, 83.6)
- moved kibuzzard-65D460A0 0.39 mm to (123.7, 88.5)
- moved kibuzzard-65D46066 0.38 mm to (123.7, 86.0)
Connections:
- J1 pad 1: +3.3V -> GND
- J1 pad 2: GND -> +3.3V
- U3 pad 13: LO6 -> LI3
- U3 pad 14: LO7 -> LO6
- U3 pad 15: LI3 -> LO7
Routing:
- net +3.3V: track 11.5 -> 81.5 mm, vias 2 -> 12
- net GND: track 0.00 -> 35.6 mm, vias 0 -> 46
- net HI2: track 2.16 -> 26.8 mm, vias 0 -> 2
- net LI3: track 4.04 -> 27.8 mm
- net HI1: track 2.28 -> 24.3 mm, vias 0 -> 2
- net HO1: track 0.00 -> 18.4 mm, vias 0 -> 4
- net HO2: track 0.00 -> 16.3 mm, vias 0 -> 2
- net Net-(U3-GPIO2/ADC1_CH2): track 38.0 -> 28.0 mm, vias 1 -> 3
- net Net-(U3-GPIO8): track 0.00 -> 9.83 mm, vias 0 -> 1
- net TX: track 0.00 -> 8.36 mm
- net +VDC: track 0.00 -> 5.88 mm, vias 0 -> 4
- net /SW: track 0.00 -> 5.31 mm
- net RX: track 0.00 -> 5.28 mm
- net /VIN_P: track 0.00 -> 4.58 mm
- net /FB: track 0.00 -> 3.08 mm
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- added copper zone on B.Cu, net +3.3V
- added copper zone on F.Cu, net +3.3V
- added copper zone on F.Cu, net +VDC
- added copper zone on F.Cu, net /VIN_P
