File: CAD/uplc/uplc.kicad_pcb (KiCad board)
At the start: 4 copper layers, 31.4 x 21 mm, 53 parts, among them J1 Conn_01x06_Pin, J2 SM12B-GHS-TB(LF)(SN), K1 G6K-2F-Y, K2 G6K-2F-Y, U1 AP63201WU, U2 TBD62003AFWG, U3 ESP32-C3-WROOM-02, Y1 32.768khz 3215 12.5pf

Commit message: Panelization changes
Routing:
- added copper zone on In1.Cu, net +3.3V
- added copper zone on In1.Cu, net HO1
- added copper zone on In1.Cu, net HO2
- removed copper zone on In2.Cu, net +3.3V
- removed copper zone on In2.Cu, net HO1
- removed copper zone on In2.Cu, net HO2
Other:
- board size 31.4 x 21 mm -> 31.4 x 22 mm

Commit message: Rev 1.2
Parts:
- L1: value 6.8uH -> 4.7uH
