File: CAD/uplc/uplc.kicad_sch (KiCad schematic)
At the start: 34 parts, among them J1 Conn_01x06_Pin, J2 SM12B-GHS-TB(LF)(SN), K1 G6K-2F-Y, K2 G6K-2F-Y, U1 DS8242-33S5, U3 ESP32-C3-WROOM-02, U5 TBD62003AFWG, Y1 32.568khz

Commit message: Value updates
Parts:
- U3: LCSC Part # (none) -> C2934560
- Y1: value 32.568khz -> 32.568khz 3.2x1.5 12.5pf
Other:
- moved on the sheet: C1, C4
Changed lines of the file:
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@@
     (stroke (width 0) (type default))
   )
-  (wire (pts (xy 46.99 40.64) (xy 49.53 40.64))
+  (wire (pts (xy 43.18 40.64) (xy 49.53 40.64))
     (stroke (width 0) (type default))
   )
@@
     (stroke (width 0) (type default))
   )
-  (wire (pts (xy 46.99 48.26) (xy 49.53 48.26))
+  (wire (pts (xy 43.18 48.26) (xy 49.53 48.26))
     (stroke (width 0) (type default))
   )
@@
     )
   )
-  (symbol (lib_id "power:GND") (at 39.37 48.26 270) (unit 1)
+  (symbol (lib_id "power:GND") (at 35.56 48.26 270) (unit 1)
     (in_bom yes) (on_board yes) (dnp no)
-    (property "Reference" "#PWR010" (at 33.02 48.26 0)
-      (effects (font (size 1.27 1.27)) hide)
-    )
-    (property "Value" "GND" (at 35.56 48.26 0)
-      (effects (font (size 1.27 1.27)))
-    )
-    (property "Footprint" "" (at 39.37 48.26 0)
-      (effects (font (size 1.27 1.27)) hide)
-    )
-    (property "Datasheet" "" (at 39.37 48.26 0)
+    (property "Reference" "#PWR010" (at 29.21 48.26 0)
+      (effects (font (size 1.27 1.27)) hide)
+    )
+    (property "Value" "GND" (at 31.75 48.26 0)
+      (effects (font (size 1.27 1.27)))
+    )
+    (property "Footprint" "" (at 35.56 48.26 0)
+      (effects (font (size 1.27 1.27)) hide)
+    )
+    (property "Datasheet" "" (at 35.56 48.26 0)
       (effects (font (size 1.27 1.27)) hide)
     )
@@
     (property "TEST" "" (at 92.71 53.34 0)
       (effects (font (size 1.27 1.27)))
+    )
+    (property "LCSC Part #" "C2934560" (at 92.71 53.34 0)
+      (effects (font (size 1.27 1.27)) hide)
     )
     (pin "1")
@@
     )
   )
-  (symbol (lib_id "Library:C") (at 43.18 48.26 270) (unit 1)
-    (in_bom yes) (on_board yes) (dnp no) (fields_autoplaced)
-    (property "Reference" "C4" (at 44.45 52.07 0)
-      (effects (font (size 1.27 1.27)) (justify left))
-    )
-    (property "Value" "20pf" (at 41.91 52.07 0)
-      (effects (font (size 1.27 1.27)) (justify left))
-    )
-    (property "Footprint" "Capacitor_SMD:C_0402_1005Metric" (at 39.37 49.2252 0)
-      (effects (font (size 1.27 1.27)) hide)
-    )
-    (property "Datasheet" "~" (at 43.18 48.26 0)
-      (effects (font (size 1.27 1.27)) hide)
-    )
-    (property "LCSC Part #" "C1554" (at 43.18 48.26 0)
-      (effects (font (size 1.27 1.27)) hide)
-    )
-    (property "TEST" "" (at 43.18 48.26 0)
+  (symbol (lib_id "Library:C") (at 39.37 48.26 270) (unit 1)
+    (in_bom yes) (on_board yes) (dnp no) (fields_autoplaced)
+    (property "Reference" "C4" (at 40.64 52.07 0)
+      (effects (font (size 1.27 1.27)) (justify left))
+    )
+    (property "Value" "20pf" (at 38.1 52.07 0)
+      (effects (font (size 1.27 1.27)) (justify left))
+    )
+    (property "Footprint" "Capacitor_SMD:C_0402_1005Metric" (at 35.56 49.2252 0)
+      (effects (font (size 1.27 1.27)) hide)
+    )
+    (property "Datasheet" "~" (at 39.37 48.26 0)
+      (effects (font (size 1.27 1.27)) hide)
+    )
+    (property "LCSC Part #" "C1554" (at 39.37 48.26 0)
+      (effects (font (size 1.27 1.27)) hide)
+    )
+    (property "TEST" "" (at 39.37 48.26 0)
       (effects (font (size 1.27 1.27)))
     )
@@
     )
   )
-  (symbol (lib_id "power:GND") (at 39.37 40.64 270) (unit 1)
-    (in_bom yes) (on_board yes) (dnp no) (fields_autoplaced)
-    (property "Reference" "#PWR09" (at 33.02 40.64 0)
-      (effects (font (size 1.27 1.27)) hide)
-    )
-    (property "Value" "GND" (at 35.56 40.64 0)
-      (effects (font (size 1.27 1.27)))
-    )
-    (property "Footprint" "" (at 39.37 40.64 0)
-      (effects (font (size 1.27 1.27)) hide)
-    )
-    (property "Datasheet" "" (at 39.37 40.64 0)
+  (symbol (lib_id "power:GND") (at 35.56 40.64 270) (unit 1)
+    (in_bom yes) (on_board yes) (dnp no) (fields_autoplaced)
+    (property "Reference" "#PWR09" (at 29.21 40.64 0)
+      (effects (font (size 1.27 1.27)) hide)
+    )
+    (property "Value" "GND" (at 31.75 40.64 0)
+      (effects (font (size 1.27 1.27)))
+    )
+    (property "Footprint" "" (at 35.56 40.64 0)
+      (effects (font (size 1.27 1.27)) hide)
+    )
+    (property "Datasheet" "" (at 35.56 40.64 0)
       (effects (font (size 1.27 1.27)) hide)
     )
@@
     )
   )
-  (symbol (lib_id "Library:C") (at 43.18 40.64 90) (unit 1)
-    (in_bom yes) (on_board yes) (dnp no) (fields_autoplaced)
-    (property "Reference" "C1" (at 41.91 36.83 0)
-      (effects (font (size 1.27 1.27)) (justify left))
-    )
-    (property "Value" "20pf" (at 44.45 36.83 0)
-      (effects (font (size 1.27 1.27)) (justify left))
-    )
-    (property "Footprint" "Capacitor_SMD:C_0402_1005Metric" (at 46.99 39.6748 0)
-      (effects (font (size 1.27 1.27)) hide)
-    )
-    (property "Datasheet" "~" (at 43.18 40.64 0)
-      (effects (font (size 1.27 1.27)) hide)
-    )
-    (property "LCSC Part #" "C1554" (at 43.18 40.64 0)
-      (effects (font (size 1.27 1.27)) hide)
-    )
-    (property "TEST" "" (at 43.18 40.64 0)
+  (symbol (lib_id "Library:C") (at 39.37 40.64 90) (unit 1)
+    (in_bom yes) (on_board yes) (dnp no) (fields_autoplaced)
+    (property "Reference" "C1" (at 38.1 36.83 0)
+      (effects (font (size 1.27 1.27)) (justify left))
+    )
+    (property "Value" "20pf" (at 40.64 36.83 0)
+      (effects (font (size 1.27 1.27)) (justify left))
+    )
+    (property "Footprint" "Capacitor_SMD:C_0402_1005Metric" (at 43.18 39.6748 0)
+      (effects (font (size 1.27 1.27)) hide)
+    )
+    (property "Datasheet" "~" (at 39.37 40.64 0)
+      (effects (font (size 1.27 1.27)) hide)
+    )
+    (property "LCSC Part #" "C1554" (at 39.37 40.64 0)
+      (effects (font (size 1.27 1.27)) hide)
+    )
+    (property "TEST" "" (at 39.37 40.64 0)
       (effects (font (size 1.27 1.27)))
     )
@@
       (effects (font (size 1.27 1.27)) (justify right))
     )
-    (property "Value" "32.568khz" (at 47.7327 49.9679 90)
+    (property "Value" "32.568khz 3.2x1.5 12.5pf" (at 41.667 49.8894 90)
       (effects (font (size 1.27 1.27)) (justify right))
     )

Commit message: rev 1.1
Parts:
- removed U1: DS8242-33S5, Package_TO_SOT_SMD:SOT-23-5, symbol Library:DS8242
- removed U5: TBD62003AFWG, Package_SO:SOIC-16_3.9x9.9mm_P1.27mm, symbol Library:ULN2003A
- added C12, C8: 22uf, Capacitor_SMD:C_0402_1005Metric, symbol Library:C
- added D4: 1N5819WS, Diode_SMD:D_SOD-323, symbol Library:1N4148WS
- added L1: 6.8uH, Inductor_SMD:L_1008_2520Metric, symbol Device:L
- added R14: 182k, Resistor_SMD:R_0402_1005Metric, symbol Library:R
- added R15: 62k, Resistor_SMD:R_0402_1005Metric, symbol Library:R
- added U1: AP63201WU, Package_TO_SOT_SMD:TSOT-23-6, symbol Regulator_Switching:AP63201WU
- added U2: ULN2803QN, Package_DFN_QFN:QFN-20-1EP_4x4mm_P0.5mm_EP2.6x2.6mm, symbol Library:ULN2803QN
- C11: value 1uF -> 22uf; LCSC Part # C52923 -> C415703
- C2: value 1uF -> 0.1uF; LCSC Part # C52923 -> C307331
- C5: value 0.1uF -> 4.7uF; footprint Capacitor_SMD:C_0402_1005Metric -> Capacitor_SMD:C_0603_1608Metric
- C7: value 1uF -> 4.7uF; footprint Capacitor_SMD:C_0402_1005Metric -> Capacitor_SMD:C_0603_1608Metric; LCSC Part # C52923 -> C307331
Connections:
- net +3.3V: now also C12.1, C8.1, L1.2, R14.2; no longer C7.1
- net +VDC: now also D4.2 (A); no longer C2.1, C5.2, R6.1
- net GND: now also C5.2, C12.2, C8.2, R15.1, U1.4 (GND), U2.21 (PAD), U2.8 (GND); no longer C2.2, C5.1, C9.2
- net HI1: now also U2.5 (I7)
- net HI2: now also U2.6 (I8)
- net HO1: now also U2.16 (O2), U2.17 (O1)
- net HO2: now also U2.14 (O4), U2.15 (O3)
- net LI12: now also U2.19 (I1), U2.20 (I2)
- net LI3: now also U2.1 (I3), U2.2 (I4)
- net LI4: now also U3.5 (GPIO6), U2.3 (I5); no longer U3.4 (GPIO5/ADC2_CH0)
- net LI5: now also U3.4 (GPIO5/ADC2_CH0), U2.4 (I6); no longer U3.5 (GPIO6)
- net LO6: now also U2.11 (O7)
- net LO7: now also U2.10 (O8)
- net RO1: now also U2.12 (O6)
- net RO2: now also U2.13 (O5)
- new net: C2.2, U1.6 (BST)
- new net FB: C9.2, R14.1, R15.2, U1.1 (FB)
- new net SW: C2.1, L1.1, U1.5 (SW)
- new net VIN_P: C5.1, C7.1, D4.1 (K), R6.1, U1.2 (EN), U1.3 (IN)
- no-connect marks 2 -> 1
Other:
- moved on the sheet: J2, R10, R11, R12, R7, R8, R9

Commit message: Rev 1.2
Parts:
- removed C10, C6: 0.1uF, Capacitor_SMD:C_0402_1005Metric, symbol Library:C
- removed C7: 4.7uF, Capacitor_SMD:C_0603_1608Metric, symbol Library:C
- removed D3: 1N5819WS, Diode_SMD:D_SOD-323, symbol Library:1N4148WS
- removed R13: 1M, Resistor_SMD:R_0402_1005Metric, symbol Library:R
- removed R3: 13.7k, Resistor_SMD:R_0402_1005Metric, symbol Library:R
- removed R6: 316k, Resistor_SMD:R_0402_1005Metric, symbol Library:R
- removed U2: ULN2803QN, Package_DFN_QFN:QFN-20-1EP_4x4mm_P0.5mm_EP2.6x2.6mm, symbol Library:ULN2803QN
- added U2: TBD62003AFWG, Package_SO:SOIC-16_3.9x9.9mm_P1.27mm, symbol esprelay:ULN2003A
- C5: value 4.7uF -> 10uF; footprint Capacitor_SMD:C_0603_1608Metric -> Capacitor_SMD:C_0805_2012Metric; LCSC Part # C307331 -> (none)
Connections:
- net GND: now also U2.8 (GND)
- net HI1: now also U2.5 (I5)
- net HI2: now also U2.6 (I6)
- net HO1: now also U2.15 (O2), U2.16 (O1)
- net HO2: now also U2.14 (O3)
- net LI12: now also U2.1 (I1), U2.2 (I2)
- net LI3: now also U2.3 (I3)
- net LI4: now also U2.4 (I4)
- net LI5: now also U2.7 (I7)
- net LO6: now also U2.12 (O5)
- net LO7: now also U2.11 (O6)
- net RO1: now also U2.10 (O7)
- net RO2: now also U2.13 (O4)
Other:
- note removed: "30v-1v vdiv"
- note removed: "Voltage sensor"
- moved on the sheet: R1

Commit message: Production push rev 1.2
Parts:
- C5: LCSC Part # (none) -> C162422
- J1: LCSC Part # (none) -> DNP
- L1: LCSC Part # (none) -> C98340
- R14: LCSC Part # (none) -> C11481
- R15: LCSC Part # (none) -> C137950
- U1: LCSC Part # (none) -> C2071044
- Y1: value 32.568khz 3.2x1.5 12.5pf -> 32.768khz 3215 12.5pf
Connections:
- net +3.3V: now also J1.2 (Pin_2); no longer J1.1 (Pin_1)
- net GND: now also J1.1 (Pin_1); no longer J1.2 (Pin_2)
- net LI3: now also U3.13 (GPIO18/USB_D-); no longer U3.15 (GPIO3/ADC1_CH3)
- net LO6: now also U3.14 (GPIO19/USB_D+); no longer U3.13 (GPIO18/USB_D-)
- net LO7: now also U3.15 (GPIO3/ADC1_CH3); no longer U3.14 (GPIO19/USB_D+)
Changed lines of the file:
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@@
     )
   )
-  (global_label "LO7" (shape input) (at 120.65 45.72 0) (fields_autoplaced)
-    (effects (font (size 1.27 1.27)) (justify left))
-    (property "Intersheetrefs" "${INTERSHEET_REFS}" (at 129.32 45.72 0)
+  (global_label "LO7" (shape input) (at 120.65 53.34 0) (fields_autoplaced)
+    (effects (font (size 1.27 1.27)) (justify left))
+    (property "Intersheetrefs" "${INTERSHEET_REFS}" (at 129.32 53.34 0)
       (effects (font (size 1.27 1.27)) (justify left) hide)
     )
@@
     )
   )
-  (global_label "LI3" (shape input) (at 120.65 53.34 0) (fields_autoplaced)
-    (effects (font (size 1.27 1.27)) (justify left))
-    (property "Intersheetrefs" "${INTERSHEET_REFS}" (at 130.5295 53.34 0)
+  (global_label "LI3" (shape input) (at 120.65 43.18 0) (fields_autoplaced)
+    (effects (font (size 1.27 1.27)) (justify left))
+    (property "Intersheetrefs" "${INTERSHEET_REFS}" (at 130.5295 43.18 0)
       (effects (font (size 1.27 1.27)) (justify left) hide)
     )
@@
     )
   )
-  (global_label "LO6" (shape input) (at 120.65 43.18 0) (fields_autoplaced)
-    (effects (font (size 1.27 1.27)) (justify left))
-    (property "Intersheetrefs" "${INTERSHEET_REFS}" (at 129.32 43.18 0)
+  (global_label "LO6" (shape input) (at 120.65 45.72 0) (fields_autoplaced)
+    (effects (font (size 1.27 1.27)) (justify left))
+    (property "Intersheetrefs" "${INTERSHEET_REFS}" (at 129.32 45.72 0)
       (effects (font (size 1.27 1.27)) (justify left) hide)
     )
@@
       (effects (font (size 1.27 1.27)) hide)
     )
-    (property "LCSC Part #" "" (at 85.09 125.73 0)
+    (property "LCSC Part #" "C137950" (at 85.09 125.73 0)
       (effects (font (size 1.27 1.27)) hide)
     )
@@
     )
   )
-  (symbol (lib_id "power:+3.3V") (at 176.53 44.45 270) (unit 1)
-    (in_bom yes) (on_board yes) (dnp no) (fields_autoplaced)
-    (property "Reference" "#PWR033" (at 172.72 44.45 0)
-      (effects (font (size 1.27 1.27)) hide)
-    )
-    (property "Value" "+3.3V" (at 180.34 44.45 90)
-      (effects (font (size 1.27 1.27)) (justify left))
-    )
-    (property "Footprint" "" (at 176.53 44.45 0)
-      (effects (font (size 1.27 1.27)) hide)
-    )
-    (property "Datasheet" "" (at 176.53 44.45 0)
+  (symbol (lib_id "power:+3.3V") (at 176.53 46.99 270) (unit 1)
+    (in_bom yes) (on_board yes) (dnp no) (fields_autoplaced)
+    (property "Reference" "#PWR033" (at 172.72 46.99 0)
+      (effects (font (size 1.27 1.27)) hide)
+    )
+    (property "Value" "+3.3V" (at 180.34 46.99 90)
+      (effects (font (size 1.27 1.27)) (justify left))
+    )
+    (property "Footprint" "" (at 176.53 46.99 0)
+      (effects (font (size 1.27 1.27)) hide)
+    )
+    (property "Datasheet" "" (at 176.53 46.99 0)
       (effects (font (size 1.27 1.27)) hide)
     )
@@
       (effects (font (size 1.27 1.27)))
     )
+    (property "LCSC Part #" "C98340" (at 73.66 113.03 0)
+      (effects (font (size 1.27 1.27)) hide)
+    )
     (pin "1")
     (pin "2")
@@
     )
     (property "Datasheet" "https://www.diodes.com/assets/Datasheets/AP63200-AP63201-AP63203-AP63205.pdf" (at 48.26 115.57 0)
+      (effects (font (size 1.27 1.27)) hide)
+    )
+    (property "LCSC Part #" "C2071044" (at 48.26 115.57 0)
       (effects (font (size 1.27 1.27)) hide)
     )
@@
     )
   )
-  (symbol (lib_id "power:GND") (at 176.53 46.99 90) (unit 1)
-    (in_bom yes) (on_board yes) (dnp no)
-    (property "Reference" "#PWR034" (at 182.88 46.99 0)
-      (effects (font (size 1.27 1.27)) hide)
-    )
-    (property "Value" "GND" (at 180.34 46.99 90)
+  (symbol (lib_id "power:GND") (at 176.53 44.45 90) (unit 1)
+    (in_bom yes) (on_board yes) (dnp no)
+    (property "Reference" "#PWR034" (at 182.88 44.45 0)
+      (effects (font (size 1.27 1.27)) hide)
+    )
+    (property "Value" "GND" (at 180.34 44.45 90)
       (effects (font (size 1.27 1.27)) (justify right))
     )
-    (property "Footprint" "" (at 176.53 46.99 0)
-      (effects (font (size 1.27 1.27)) hide)
-    )
-    (property "Datasheet" "" (at 176.53 46.99 0)
+    (property "Footprint" "" (at 176.53 44.45 0)
+      (effects (font (size 1.27 1.27)) hide)
+    )
+    (property "Datasheet" "" (at 176.53 44.45 0)
       (effects (font (size 1.27 1.27)) hide)
     )
@@
       (effects (font (size 1.27 1.27)) hide)
     )
-    (property "LCSC Part #" "" (at 171.45 49.53 0)
+    (property "LCSC Part #" "DNP" (at 171.45 49.53 0)
       (effects (font (size 1.27 1.27)) hide)
     )
@@
       (effects (font (size 1.27 1.27)) hide)
     )
-    (property "LCSC Part #" "" (at 22.86 116.84 0)
+    (property "LCSC Part #" "C162422" (at 22.86 116.84 0)
       (effects (font (size 1.27 1.27)) hide)
     )
@@
       (effects (font (size 1.27 1.27)) (justify right))
     )
-    (property "Value" "32.568khz 3.2x1.5 12.5pf" (at 41.667 49.8894 90)
+    (property "Value" "32.768khz 3215 12.5pf" (at 41.667 49.8894 90)
       (effects (font (size 1.27 1.27)) (justify right))
     )
@@
       (effects (font (size 1.27 1.27)) hide)
     )
-    (property "Datasheet" "~" (at 49.53 44.45 0)
+    (property "Datasheet" "https://datasheet.lcsc.com/lcsc/1810171817_Seiko-Epson-Q13FC1350000400_C32346.pdf" (at 49.53 44.45 0)
       (effects (font (size 1.27 1.27)) hide)
     )
@@
       (effects (font (size 1.27 1.27)) hide)
     )
-    (property "LCSC Part #" "" (at 85.09 116.84 0)
-      (effects (font (size 1.27 1.27)) hide)
-    )
+    (property "LCSC Part #" "C11481" (at 85.09 116.84 0)
+      (effects (font (size 1.27 1.27)) hide)
+    )
