File: CAD/uplc/uplc.kicad_sch (KiCad schematic)
At the start: 33 parts, among them J1 Conn_01x06_Pin, J2 SM12B-GHS-TB(LF)(SN), K1 G6K-2F-Y, K2 G6K-2F-Y, U1 AP63201WU, U2 TBD62003AFWG, U3 ESP32-C3-WROOM-02, Y1 32.768khz 3215 12.5pf

Commit message: Rev 1.2
Parts:
- C1, C4: Generic (none) -> x; MPN (none) -> 0402CG200J500NT
- C11, C12, C8: Generic (none) -> x; MPN (none) -> GRM155R60J226ME11D
- C2, C3, C9: Generic (none) -> x; LCSC Part # C307331 -> C77020; MPN (none) -> GRM155R71H104KE14D
- C5: Generic (none) -> x; MPN (none) -> GRM21BR6YA106KE43L
- D1, D2, D4: MPN (none) -> 1N5819WS
- J2: MPN (none) -> SM12B-GHS-TB(LF)(SN)
- K1, K2: LCSC Part # C2982926 -> C93168; MPN (none) -> G6K-2F-Y DC3
- L1: value 6.8uH -> 4.7uH; Generic (none) -> x; LCSC Part # C98340 -> C82314; MPN (none) -> LQM2HPN4R7MG0L
- R1, R10, R11, R12, R2, R4, R5, R7, R8, R9: Generic (none) -> x; MPN (none) -> 0402WGF1002TCE
- R14: Generic (none) -> x; MPN (none) -> 0402WGF1823TCE
- R15: Generic (none) -> x; MPN (none) -> RC0402FR-0762KL
- U1: MPN (none) -> AP63201WU-7
- U2: MPN (none) -> TBD62003AFWG
- U3: MPN (none) -> ESP32-C3-WROOM-02-N4
- Y1: MPN (none) -> Q13FC13500004
